Commit message: 240220_2035

File: ackermann_vehicle_description/urdf/em_3905.urdf.xacro (robot description, xacro)
@@ -344,4 +344,32 @@
     <child link="chassis"/>
   </joint>
+  <!-- Roof -->
+  <link name="roof">
+    <visual>
+      <origin xyz="-0.064 0 0.07"/>
+      <geometry>
+        <box size="0.192 ${chassis_width} 0.14"/>
+      </geometry>
+      <material name="chassis_mat"/>
+    </visual>
+    <collision>
+      <origin xyz="0 0 0.07"/>
+      <geometry>
+        <box size="${chassis_length} ${chassis_width} 0.14"/>
+      </geometry>
+    </collision>
+    <xacro:solid_cuboid_inertial
+        width="${chassis_length}" depth="${chassis_width}"
+        height="0.14" mass="${chassis_mass}">
+      <origin xyz="0 0 0.07"/>
+    </xacro:solid_cuboid_inertial>
+  </link>
+  <gazebo reference="chassis">
+    <material>Gazebo/Grey</material>
+  </gazebo>
+  <joint name="chassis_to_roof" type="fixed">
+    <parent link="chassis"/>
+    <child link="roof"/>
+  </joint>
   <!-- Batteries -->
   <xacro:battery prefix="left" reflect="1"/>
@@ -359,7 +387,7 @@
     <plugin name="gazebo_ros_control" filename="libgazebo_ros_control.so"/>
   </gazebo>
-  <xacro:arg name="camera_visual" default="false"/>
+  <xacro:arg name="camera_visual" default="true"/>
   <joint name="camera_joint" type="fixed">
-    <origin xyz="0.073 -0.011 0.084" rpy="0 0 0"/>
+    <origin xyz="-0.173 -0.011 0.200" rpy="0 -0.05 0"/>
     <parent link="base_link"/>
     <child link="camera_link"/>
@@ -398,5 +426,5 @@
           <clip>
               <near>0.03</near>
-              <far>100</far>
+              <far>500</far>
           </clip>
       </camera>

Commit message: 240228_0654

File: ackermann_vehicle_description/urdf/em_3905.urdf.xacro (robot description, xacro)
@@ -389,5 +389,5 @@
   <xacro:arg name="camera_visual" default="true"/>
   <joint name="camera_joint" type="fixed">
-    <origin xyz="-0.173 -0.011 0.200" rpy="0 -0.05 0"/>
+    <origin xyz="-0.173 0.000 0.200" rpy="0 -0.05 0"/>
     <parent link="base_link"/>
     <child link="camera_link"/>
@@ -395,5 +395,5 @@
   <link name="camera_link">
     <collision>
-      <origin xyz="0.005 0.011 0.013" rpy="0 0 0"/>
+      <origin xyz="0.005 0.000 0.013" rpy="0 0 0"/>
       <geometry>
         <box size="0.015 0.030 0.027"/>
@@ -402,5 +402,5 @@
   </link>
   <joint name="camera_rgb_joint" type="fixed">
-    <origin xyz="0.003 0.011 0.009" rpy="0 0 0"/>
+    <origin xyz="0.003 0.000 0.009" rpy="0 0 0"/>
     <parent link="camera_link"/>
     <child link="camera_rgb_frame"/>
